File: PCB/Joy Controller V2.kicad_pcb (KiCad board)
At the start: 2 copper layers, 172.6 x 66.7 mm, 23 parts, among them J1 Conn_02x16_Odd_Even, J2 JOY1, J3 JOY2, J4 USB_C_Receptacle_USB2.0_16P, SW1 SW_Push, SW10 SW_Push, SW11 SW_Push, SW2 SW_Push, SW3 SW_Push, SW4 SW_Push, SW5 SW_Push, SW6 SW_Push, SW7 SW_Push, SW8 SW_Push, SW9 SW_Push

Commit message: Add files via upload
Parts:
- removed SW11, SW9: SW_Push, Button_Switch_THT:SW_Tactile_SKHH_Angled
- added JP1: SolderJumper_2_Bridged, Jumper:SolderJumper-2_P1.3mm_Open_RoundedPad1.0x1.5mm, F.Cu at (174.0, 70.0)
- added JP2: SolderJumper_2_Bridged, Jumper:SolderJumper-2_P1.3mm_Open_RoundedPad1.0x1.5mm, F.Cu at (174.0, 75.0)
- added SW12: RotaryEncoder_Switch_MP, Rotary_Encoder:RotaryEncoder_Alps_EC11E-Switch_Vertical_H20mm_MountingHoles, F.Cu at (178.0, 70.0)
- moved SW7 4.93 mm to (54.0, 121.7)
- moved J2 4.93 mm to (82.3, 75.0)
- moved SW5 4.93 mm to (54.1, 97.7)
- moved SW6 4.93 mm to (66.0, 109.7)
- moved SW8 4.93 mm to (42.1, 109.7)
- moved J3 4.90 mm to (175.5, 122.0)
- moved SW1 4.90 mm to (197.3, 71.0)
- moved SW2 4.90 mm to (209.2, 83.0)
- moved SW3 4.90 mm to (197.2, 95.0)
- moved SW4 4.90 mm to (185.3, 83.0)
Routing:
- net RXD(GPIO44): track 50.6 -> 117.7 mm
- net TXD(GPIO43): track 56.5 -> 119.1 mm
- net RST: track 59.6 -> 0.00 mm
- net GPIO38: track 67.5 -> 103.9 mm, vias 1 -> 2
- net GPIO39: track 122.1 -> 128.5 mm
- net GPIO42: track 92.9 -> 97.8 mm
- net GPIO41: track 101.8 -> 106.7 mm
- net GPIO40: track 119.6 -> 124.4 mm
- net Net-(JP2-B): track 0.00 -> 3.37 mm
- net Net-(JP1-B): track 0.00 -> 3.32 mm
- net GPIO21: track 62.2 -> 62.8 mm
Other:
- board size 172.6 x 66.7 mm -> 182.7 x 66.7 mm

Commit message: Add files via upload
Parts:
- removed J2: JOY1, Connector_PinSocket_2.54mm:PinSocket_1x05_P2.54mm_Horizontal
- removed J3: JOY2, Connector_PinSocket_2.54mm:PinSocket_1x05_P2.54mm_Horizontal
- added JP3: SolderJumper_3_Open, Jumper:SolderJumper-3_P1.3mm_Open_RoundedPad1.0x1.5mm, F.Cu at (46.4, 42.7)
- added SW11: SW_Push, Button_Switch_THT:SW_Tactile_SKHH_Angled, F.Cu at (46.5, 67.7)
- added SW9: SW_Push, Button_Switch_THT:SW_PUSH_6mm, F.Cu at (180.3, 100.0)
- added SW9: SW_Push, Button_Switch_THT:SW_PUSH_6mm, F.Cu at (78.6, 98.0)
- added U1: COM-09032, Joy:JOYSTICK, B.Cu at (62.2, 80.9)
- added U2: COM-09032, Joy:JOYSTICK, B.Cu at (195.6, 116.2)
- JP1: value SolderJumper_2_Bridged -> SolderJumper_2_Open
- JP2: value SolderJumper_2_Bridged -> SolderJumper_3_Open; footprint Jumper:SolderJumper-2_P1.3mm_Open_RoundedPad1.0x1.5mm -> Jumper:SolderJumper-3_P1.3mm_Open_RoundedPad1.0x1.5mm
- SW12: value RotaryEncoder_Switch_MP -> SW_Push; footprint Rotary_Encoder:RotaryEncoder_Alps_EC11E-Switch_Vertical_H20mm_MountingHoles -> Button_Switch_THT:SW_Tactile_SKHH_Angled
- moved JP2 132.7 mm to (46.4, 38.9)
- moved JP1 126.6 mm to (51.4, 38.9)
- moved SW12 29.0 mm to (206.9, 67.8)
- moved SW7 4.93 mm to (59.0, 121.8)
- moved SW5 4.93 mm to (59.0, 97.8)
- moved SW6 4.93 mm to (71.0, 109.8)
- moved SW8 4.93 mm to (47.0, 109.8)
- moved SW1 4.90 mm to (192.4, 71.0)
- moved SW2 4.90 mm to (204.3, 83.0)
- moved SW3 4.90 mm to (192.3, 95.0)
- moved SW4 4.90 mm to (180.4, 83.0)
Connections:
- JP1 pad 1: RXD(GPIO44) -> Net-(JP1-A)
- JP1 pad 2: Net-(JP1-B) -> BOOT(GPIO0)
- JP2 pad 1: TXD(GPIO43) -> Net-(JP2-A)
- JP2 pad 2: Net-(JP2-B) -> RXD(GPIO44)
Routing:
- net GPIO38: track 103.9 -> 0.00 mm, vias 2 -> 0
- net RXD(GPIO44): track 117.7 -> 50.6 mm
- net TXD(GPIO43): track 119.1 -> 56.5 mm
- net GPIO41: track 106.7 -> 112.9 mm
- net GPIO42: track 97.8 -> 92.9 mm
- net Net-(JP2-B): track 3.37 -> 0.00 mm
- net Net-(JP1-B): track 3.32 -> 0.00 mm
- net GPIO39: track 128.5 -> 125.7 mm
- net GPIO10: track 67.1 -> 65.2 mm
- net GPIO11: track 57.4 -> 55.8 mm
- net GPIO9: track 70.2 -> 68.7 mm
- net GPIO21: track 62.8 -> 62.2 mm
Other:
- board size 182.7 x 66.7 mm -> 172.6 x 66.8 mm

Commit message: Add files via upload
Parts:
- removed the SW9 at (78.6, 98.0)
- added SW13: SW_Push, Button_Switch_THT:SW_PUSH_6mm, F.Cu at (72.1, 96.5)
- J4: footprint Connector_USB:USB_C_Receptacle_GCT_USB4110 -> Connector_USB:USB_C_Receptacle_GCT_USB4105-xx-A_16P_TopMnt_Horizontal
- U1, U2: moved to F.Cu
- moved JP1 144.3 mm to (180.0, 104.3), turned to -90 degrees
- moved JP2 87.8 mm to (116.7, 91.5), turned to 180 degrees
- moved JP3 79.7 mm to (114.2, 84.5), turned to 180 degrees
- moved SW9 3.45 mm to (180.3, 96.5)
- turned U1 to 90 degrees
- turned U2 to -90 degrees
Connections:
- U1 pad B1A: GPIO21 -> GPIO9
- U1 pad H2: GPIO18 -> GPIO11
- U1 pad V2: GPIO17 -> GPIO10
- U2 pad B1A: GPIO21 -> GPIO38
Routing:
- net Net-(JP2-A): track 0.00 -> 115.5 mm
- net GPIO38: track 0.00 -> 105.7 mm
- net Net-(JP3-A): track 0.00 -> 71.7 mm
- net +3.3V: track 108.6 -> 172.7 mm
- net BOOT(GPIO0): track 0.00 -> 58.3 mm
- net GPIO17: track 47.7 -> 87.1 mm
- net GPIO10: track 65.2 -> 89.8 mm, vias 1 -> 0
- net GPIO9: track 68.7 -> 93.0 mm
- net GPIO11: track 55.8 -> 77.2 mm
- net GPIO18: track 45.7 -> 60.9 mm
- net Net-(JP1-A): track 0.00 -> 9.34 mm
- net GND: track 32.2 -> 23.2 mm, vias 5 -> 1
- net GPIO21: track 62.2 -> 54.4 mm
- net RXD(GPIO44): track 50.6 -> 44.3 mm
- net RXD: track 0.00 -> 5.01 mm, vias 0 -> 1
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
Commit message: Add files via upload
Parts:
- removed JP1: SolderJumper_2_Open, Jumper:SolderJumper-2_P1.3mm_Open_RoundedPad1.0x1.5mm
- removed JP2, JP3: SolderJumper_3_Open, Jumper:SolderJumper-3_P1.3mm_Open_RoundedPad1.0x1.5mm
- added D1: D, Diode_SMD:D_SOD-323, F.Cu at (213.3, 85.0)
- added D10: D, Diode_SMD:D_SOD-323, F.Cu at (69.8, 104.2)
- added D11: D, Diode_SMD:D_SOD-323, F.Cu at (47.4, 107.0)
- added D12: D, Diode_SMD:D_SOD-323, F.Cu at (48.2, 70.4)
- added D13: D, Diode_SMD:D_SOD-323, F.Cu at (178.5, 104.5)
- added D14: D, Diode_SMD:D_SOD-323, F.Cu at (203.2, 104.5)
- added D15: D, Diode_SMD:D_SOD-323, F.Cu at (192.5, 78.0)
- added D16: D, Diode_SMD:D_SOD-323, F.Cu at (208.0, 71.1)
- added D2: D, Diode_SMD:D_SOD-323, F.Cu at (203.3, 98.6)
- added D3: D, Diode_SMD:D_SOD-323, F.Cu at (189.4, 84.8)
- added D4: D, Diode_SMD:D_SOD-323, F.Cu at (201.4, 73.1)
- added D5: D, Diode_SMD:D_SOD-323, F.Cu at (79.9, 110.9)
- added D6: D, Diode_SMD:D_SOD-323, F.Cu at (68.0, 121.7)
- added D7: D, Diode_SMD:D_SOD-323, F.Cu at (44.4, 109.9)
- added D8: D, Diode_SMD:D_SOD-323, F.Cu at (68.0, 100.8)
- added D9: D, Diode_SMD:D_SOD-323, F.Cu at (95.3, 68.0)
- added R3: 10K, Resistor_SMD:R_0603_1608Metric, F.Cu at (183.2, 112.3)
- added R4: 10K, Resistor_SMD:R_0603_1608Metric, F.Cu at (56.0, 100.8)
- added R5: 10K, Resistor_SMD:R_0603_1608Metric, F.Cu at (72.8, 87.0)
- added R6: 10K, Resistor_SMD:R_0603_1608Metric, F.Cu at (178.5, 109.2)
- added R7: 10K, Resistor_SMD:R_0603_1608Metric, F.Cu at (133.2, 92.4)
- added R8: 10K, Resistor_SMD:R_0603_1608Metric, F.Cu at (137.0, 98.8)
- added SW13: SW_Push, Button_Switch_THT:SW_Tactile_SKHH_Angled, F.Cu at (98.7, 67.8)
- added SW14: RotaryEncoder_Switch_MP, Rotary_Encoder:RotaryEncoder_Alps_EC11E-Switch_Vertical_H20mm, F.Cu at (189.3, 74.9)
- moved H8 0.10 mm to (93.6, 122.8)
- moved H13 0.10 mm to (165.6, 122.8)
- moved H7 0.09 mm to (165.6, 74.2)
- renumbered H13 to H1, H11 to H13, H12 to H14, H14 to H2, H9 to H7, H10 to H8, J4 to J1, J1 to J2, SW2 to SW1, SW13 to SW10, SW12 to SW11, SW11 to SW12, SW10 to SW15, SW3 to SW2, SW4 to SW3, SW1 to SW4, SW6 to SW5, SW7 to SW6, SW8 to SW7, SW5 to SW8
Connections:
- J2 pad 9: GPIO39 -> EC11+
- SW1 pad 1: GND -> Net-(D1-A)
- SW1 pad 2: GPIO40 -> GPIO42
- SW10 pad 1: GND -> Net-(D10-A)
- SW10 pad 2: GPIO21 -> GPIO40
- SW11 pad 1: GND -> Net-(D16-A)
- SW11 pad 2: Net-(JP2-A) -> EC11+
- SW12 pad 1: GND -> Net-(D12-A)
- SW12 pad 2: Net-(JP3-A) -> GPIO40
- SW2 pad 1: GND -> Net-(D2-A)
- SW2 pad 2: GPIO41 -> GPIO42
- SW3 pad 1: GND -> Net-(D3-A)
- SW4 pad 1: GND -> Net-(D4-A)
- SW4 pad 2: GPIO39 -> GPIO42
- SW5 pad 1: GND -> Net-(D5-A)
- SW5 pad 2: GPIO47 -> GPIO41
- SW6 pad 1: GND -> Net-(D6-A)
- SW6 pad 2: GPIO46 -> GPIO41
- SW7 pad 1: GND -> Net-(D7-A)
- SW7 pad 2: GPIO48 -> GPIO41
- SW8 pad 1: GND -> Net-(D8-A)
- SW8 pad 2: GPIO45 -> GPIO41
- SW9 pad 1: GND -> Net-(D13-A)
- SW9 pad 2: Net-(JP1-A) -> EC11+
- U1 pad B1A: GPIO9 -> GPIO40
- U1 pad B2A: GND -> JOY_SW_L-
- U2 pad B1A: GPIO38 -> EC11+
- U2 pad B2A: GND -> JOY_SW_R-
Routing:
- net EC11+: track 0.00 -> 230.0 mm
- net GPIO45: track 83.9 -> 244.4 mm, vias 1 -> 2
- net GPIO47: track 73.9 -> 216.9 mm, vias 1 -> 2
- net GPIO48: track 101.0 -> 235.0 mm, vias 1 -> 2
- net GPIO39: track 125.5 -> 0.00 mm, vias 1 -> 0
- net Net-(JP2-A): track 115.5 -> 0.00 mm
- net GPIO46: track 78.7 -> 185.8 mm
- net GPIO38: track 105.7 -> 0.00 mm
- net GPIO42: track 94.3 -> 167.7 mm
- net Net-(JP3-A): track 71.7 -> 0.00 mm
- net GPIO21: track 54.4 -> 118.1 mm
- net BOOT(GPIO0): track 58.3 -> 0.00 mm
- net GPIO40: track 124.7 -> 175.0 mm, vias 1 -> 0
- net +3.3V: track 172.7 -> 200.8 mm, vias 1 -> 3
- net JOY_SW_L-: track 0.00 -> 26.1 mm, vias 0 -> 1
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Other:
- board text added: "+3.3V"
- board text added: "+5V"
- board text added: "+BATT"
- board text added: "CHG STATUS"
- board text added: "GND"
- board text added: "I2C"
- board text added: "Joy Controller V2 Merlin2LmmL"
- board text added: "PWR STATUS"
- board text added: "RXD"
- board text added: "SCL"
- board text added: "SDA"
- board text added: "TXD"
- board text added: "UART"

Commit message: Add files via upload
Parts:
- added C1: 1uF, Capacitor_SMD:C_0603_1608Metric, F.Cu at (48.9, 96.6)
- added C2: 100nF, Capacitor_SMD:C_0603_1608Metric, F.Cu at (48.9, 95.0)
- added C3: 1uF, Capacitor_SMD:C_0603_1608Metric, F.Cu at (210.6, 96.6)
- added C4: 100nF, Capacitor_SMD:C_0603_1608Metric, F.Cu at (210.6, 95.0)
- added D17: 1N4148W, Diode_SMD:D_SOD-123, F.Cu at (48.9, 93.0)
- added D18: 1N4148W, Diode_SMD:D_SOD-123, F.Cu at (210.6, 93.0)
- added MOT1: LCM1027A2445F, lcsc:VIBRATING-MOTOR-SMD_WELDING, F.Cu at (48.9, 100.2)
- added MOT2: LCM1027A2445F, lcsc:VIBRATING-MOTOR-SMD_WELDING, F.Cu at (210.6, 100.2)
- added Q1: NPN, Package_TO_SOT_SMD:SOT-23, F.Cu at (52.5, 95.8)
- added Q2: NPN, Package_TO_SOT_SMD:SOT-23, F.Cu at (206.9, 95.0)
- added R10: 1K, Resistor_SMD:R_0603_1608Metric, F.Cu at (206.0, 98.6)
- added R9: 1K, Resistor_SMD:R_0603_1608Metric, F.Cu at (52.5, 99.0)
- moved D6 6.04 mm to (74.0, 121.8)
- moved D2 1.86 mm to (201.4, 98.6)
- moved D11 1.46 mm to (46.4, 105.9), turned to 90 degrees
- moved D14 1.20 mm to (202.0, 104.5)
Connections:
- J2 pad 9: EC11+ -> GPIO39
- R6 pad 2: EC11+ -> BOOT(GPIO0)
- SW11 pad 2: EC11+ -> BOOT(GPIO0)
- SW14 pad S1: EC11+ -> BOOT(GPIO0)
- SW9 pad 2: EC11+ -> BOOT(GPIO0)
- U2 pad B1A: EC11+ -> BOOT(GPIO0)
Routing:
- net EC11+: track 230.0 -> 0.00 mm
- net BOOT(GPIO0): track 0.00 -> 218.0 mm, vias 0 -> 1
- net GPIO39: track 0.00 -> 118.5 mm, vias 0 -> 1
- net GPIO38: track 0.00 -> 98.7 mm, vias 0 -> 1
- net +3.3V: track 200.8 -> 245.7 mm
- net GND: track 34.3 -> 47.8 mm, vias 2 -> 4
- net Net-(D18-A): track 0.00 -> 11.0 mm
- net Net-(D17-A): track 0.00 -> 9.90 mm
- net GPIO46: track 185.8 -> 177.1 mm
- net GPIO42: track 167.7 -> 174.5 mm
- net Net-(D6-A): track 9.46 -> 15.5 mm
- net GPIO17: track 87.3 -> 93.2 mm
- net GPIO11: track 67.2 -> 73.1 mm
- net JOY_SW_L-: track 26.1 -> 31.6 mm
- net GPIO47: track 216.9 -> 221.6 mm
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