File: PCB/Joy Controller V2.kicad_pcb (KiCad board)
At the start: 2 copper layers, 172.6 x 66.8 mm, 67 parts, among them J1 USB_C_Receptacle_USB2.0_16P, J2 Conn_02x16_Odd_Even, Q1 NPN, Q2 NPN, SW1 SW_Push, SW10 SW_Push, SW11 SW_Push, SW12 SW_Push, SW13 SW_Push, SW14 RotaryEncoder_Switch_MP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

Commit message: Add files via upload
Parts:
- removed G***: LOGO, Joy:Penguin
- added C5: 100nF, Capacitor_SMD:C_0603_1608Metric, F.Cu at (65.0, 115.6)
- added C6: 100nF, Capacitor_SMD:C_0603_1608Metric, F.Cu at (177.9, 123.2)
- added C7: 100nF, Capacitor_SMD:C_0603_1608Metric, F.Cu at (200.1, 85.7)
- added C8: 100nF, Capacitor_SMD:C_0603_1608Metric, F.Cu at (73.3, 69.3)
- added D19: WS2812B, LED_SMD:LED_WS2812B_PLCC4_5.0x5.0mm_P3.2mm, F.Cu at (182.4, 124.1)
- added D20: WS2812B, LED_SMD:LED_WS2812B_PLCC4_5.0x5.0mm_P3.2mm, F.Cu at (195.6, 85.2)
- added D21: WS2812B, LED_SMD:LED_WS2812B_PLCC4_5.0x5.0mm_P3.2mm, F.Cu at (74.9, 73.0)
- added D22: WS2812B, LED_SMD:LED_WS2812B_PLCC4_5.0x5.0mm_P3.2mm, F.Cu at (62.2, 112.0)
- moved J1 62.5 mm to (128.4, 131.2), turned to 0 degrees
- moved R1 50.1 mm to (125.7, 125.4), turned to 180 degrees
- moved R2 49.9 mm to (131.1, 125.4), turned to 0 degrees
- moved R7 32.2 mm to (122.5, 91.7), turned to -90 degrees
- moved R8 29.1 mm to (124.5, 91.7), turned to -90 degrees
- moved R5 28.7 mm to (126.8, 91.7), turned to -45 degrees
- moved R6 26.5 mm to (130.2, 92.6), turned to 180 degrees
- moved R4 26.1 mm to (128.9, 106.9)
- moved R3 25.8 mm to (127.2, 106.9)
- moved D16 23.4 mm to (52.5, 86.2), turned to 90 degrees
- moved U3 21.8 mm to (129.5, 99.3), turned to 90 degrees
- moved R11 18.3 mm to (134.7, 92.5)
- moved U4 15.2 mm to (133.0, 113.3), turned to 0 degrees
- moved H6 8.27 mm to (177.1, 130.6)
- moved D15 5.23 mm to (174.0, 80.7), turned to 180 degrees
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Connections:
- U3 pad 1: ROW0 -> M_HAP_L
- U3 pad 15: GND -> +3.3V
- U3 pad 2: ROW1 -> ROW3
- U3 pad 21: ROT_ENC_B -> unconnected-(U3-GPA0-Pad21)
- U3 pad 22: ROT_ENC_A -> COL0
- U3 pad 23: COL0 -> M_HAP_R
- U3 pad 25: M_HAP_R -> unconnected-(U3-GPA4-Pad25)
- U3 pad 26: TH1 -> ROT_ENC_A
- U3 pad 27: unconnected-(U3-GPA6-Pad27) -> ROT_ENC_B
- U3 pad 28: unconnected-(U3-GPA7-Pad28) -> LEDs
- U3 pad 3: ROW2 -> ROW0
- U3 pad 4: ROW3 -> ROW2
- U3 pad 5: COL2 -> ROW1
- U3 pad 7: M_HAP_L -> COL2
Routing:
- net +5V: track 70.5 -> 368.3 mm, vias 3 -> 0
- net Net-(D20-DOUT): track 0.00 -> 161.3 mm
- net LEDs: track 0.00 -> 86.9 mm, vias 0 -> 2
- net Net-(D21-DOUT): track 0.00 -> 82.3 mm
- net TXD(GPIO43): track 74.4 -> 0.00 mm, vias 1 -> 0
- net RXD(GPIO44): track 62.2 -> 0.00 mm, vias 1 -> 0
- net Net-(D19-DOUT): track 0.00 -> 57.8 mm, vias 0 -> 2
- net DP: track 61.4 -> 19.2 mm
- net M_HAP_L: track 113.6 -> 71.8 mm, vias 2 -> 0
- net DN: track 62.5 -> 20.8 mm
- net ROW1: track 194.2 -> 235.8 mm, vias 7 -> 4
- net ROT_ENC_A: track 46.0 -> 81.9 mm, vias 1 -> 0
- net ROT_ENC_B: track 50.2 -> 81.8 mm, vias 1 -> 0
- net ROW0: track 184.2 -> 213.3 mm
- net GPIO38: track 66.6 -> 42.0 mm, vias 0 -> 2
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Other:
- board size 172.6 x 66.8 mm -> 172.6 x 70.1 mm

Commit message: Add files via upload
Parts:
- moved R3 15.4 mm to (127.2, 91.4)
- moved R11 15.4 mm to (134.7, 77.1)
- moved R4 15.4 mm to (128.9, 91.4)
- moved R5 15.4 mm to (126.8, 76.2)
- moved R6 15.4 mm to (130.2, 77.2)
- moved R7 15.4 mm to (122.5, 76.3)
- moved R8 15.4 mm to (124.5, 76.3)
- moved U3 15.4 mm to (129.5, 83.9)
- moved D15 0.74 mm to (174.6, 81.2), turned to 90 degrees
Connections:
- U3 pad 15: +3.3V -> GND
- U3 pad 21: unconnected-(U3-GPA0-Pad21) -> ROT_ENC_B
- U3 pad 22: COL0 -> ROT_ENC_A
- U3 pad 23: M_HAP_R -> COL0
- U3 pad 25: unconnected-(U3-GPA4-Pad25) -> M_HAP_R
- U3 pad 26: ROT_ENC_A -> TH1
- U3 pad 27: ROT_ENC_B -> unconnected-(U3-GPA6-Pad27)
- U3 pad 28: LEDs -> unconnected-(U3-GPA7-Pad28)
Routing:
- net COL0: track 169.9 -> 207.9 mm
- net JOY_L_VRy: track 80.4 -> 98.8 mm
- net JOY_L_VRx: track 98.9 -> 117.3 mm
- net LEDs: track 86.9 -> 103.0 mm
- net SDA(GPIO8): track 26.4 -> 41.8 mm
- net GPIO38: track 42.0 -> 57.4 mm
- net SCL(GPIO7): track 25.2 -> 40.7 mm
- net ROW0: track 213.3 -> 200.3 mm
- net ROW1: track 235.8 -> 247.9 mm
- net +3.3V: track 275.2 -> 283.0 mm
- net M_HAP_R: track 90.5 -> 97.3 mm
- net COL1: track 129.9 -> 136.3 mm
- net COL2: track 161.6 -> 168.0 mm
- net ROW3: track 203.6 -> 209.0 mm
- net COL3: track 182.2 -> 187.4 mm
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Other:
- outline, holes or cut-outs redrawn

Commit message: Add files via upload
Parts:
- added G***: LOGO, LOGO, F.Cu at (243.9, 225.8)
- added G***: LOGO, LOGO, F.Cu at (160.4, 101.8)
- added G***: LOGO, LOGO, F.Cu at (104.2, 107.2)
- added G***: LOGO, LOGO, F.Cu at (238.5, 246.0)
- added G***: LOGO, LOGO, F.Cu at (194.2, 216.2)
- added G***: LOGO, LOGO, F.Cu at (176.6, 208.4)
- added G***: LOGO, LOGO, B.Cu at (148.6, 91.6)
- added G***: LOGO, LOGO, B.Cu at (62.4, 80.8)
- added G***: LOGO, LOGO, B.Cu at (194.8, 116.2)
- turned H7 to 0 degrees
- turned H8 to 180 degrees
Connections:
- U3 pad 15: GND -> +3.3V
- U3 pad 21: ROT_ENC_B -> unconnected-(U3-GPA0-Pad21)
- U3 pad 22: ROT_ENC_A -> COL0
- U3 pad 23: COL0 -> M_HAP_R
- U3 pad 25: M_HAP_R -> unconnected-(U3-GPA4-Pad25)
- U3 pad 26: TH1 -> ROT_ENC_A
- U3 pad 27: unconnected-(U3-GPA6-Pad27) -> ROT_ENC_B
- U3 pad 28: unconnected-(U3-GPA7-Pad28) -> LEDs
Routing:
- net GND: track 26.7 -> 19.0 mm, vias 398 -> 507
- net JOY_L_VRx: track 117.3 -> 118.3 mm
- net unconnected-(U3-GPA4-Pad25): track 0.00 -> 0.51 mm
- net M_HAP_R: track 97.3 -> 96.8 mm
Other:
- board text removed: "+3.3V"
- board text removed: "+5V"
- board text removed: "+BATT"
- board text removed: "GND"
- board text removed: "I2C"
- board text removed: "RXD"
- board text removed: "SCL"
- board text removed: "SDA"
- board text removed: "TXD"
- board text removed: "UART"

Commit message: Add files via upload
Parts:
- removed the G*** at (243.9, 225.8)
- removed the G*** at (238.5, 246.0)
- removed the G*** at (194.2, 216.2)
- removed the G*** at (176.6, 208.4)
- removed SW15: SW_Push, Button_Switch_THT:SW_Tactile_SKHH_Angled
- moved C3 14.0 mm to (224.6, 95.4)
- moved C4 14.0 mm to (224.6, 93.8)
- moved C7 14.0 mm to (214.1, 84.5)
- moved D15 14.0 mm to (188.6, 80.0)
- moved D18 14.0 mm to (224.6, 91.8)
- moved D19 14.0 mm to (196.4, 122.8)
- moved D20 14.0 mm to (209.6, 83.9)
- moved G*** 14.0 mm to (162.6, 90.4)
- moved J1 14.0 mm to (142.4, 130.0)
- moved MOT2 14.0 mm to (224.5, 99.0)
- moved R6 14.0 mm to (144.1, 75.9)
- moved SW1 14.0 mm to (218.3, 81.7)
- moved SW14 14.0 mm to (203.3, 73.7)
- moved SW2 14.0 mm to (206.3, 93.7)
- moved SW9 14.0 mm to (194.3, 95.3)
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Routing:
- net PWR: track 73.1 -> 0.00 mm, vias 2 -> 0
- net ROW0: track 200.3 -> 206.9 mm
- net ROW2: track 179.4 -> 181.6 mm
- net JOY_R_VRx: track 69.7 -> 68.1 mm
- net JOY_L_VRx: track 118.3 -> 117.1 mm
- net GND: track 19.0 -> 19.9 mm, vias 507 -> 1751
- net Net-(D13-A): track 4.27 -> 5.13 mm
- net DP: track 19.2 -> 20.0 mm
- net SDA(GPIO8): track 41.8 -> 41.0 mm
- net +3.3V: track 283.4 -> 282.6 mm
- net SCL(GPIO7): track 40.7 -> 39.9 mm
- net Net-(D20-DOUT): track 159.1 -> 159.9 mm
- net LEDs: track 103.0 -> 102.4 mm
- net GPIO38: track 57.4 -> 58.0 mm

Commit message: Add files via upload
Parts:
- moved H5 35.5 mm to (87.2, 88.8)
- moved H6 24.6 mm to (199.4, 106.2)
Changed lines of the file:
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@@
 			(net 7 "GND")
 			(pintype "passive")
+			(zone_connect 2)
 		)
 		(embedded_fonts no)
@@
 	(footprint "MountingHole:MountingHole_2mm"
 		(layer "F.Cu")
-		(at 89.55 124.255)
+		(at 87.2 88.8)
 		(descr "Mounting Hole 2mm, no annular, generated by kicad-footprint-generator mountinghole.py")
 		(tags "mountinghole")
@@
 	(footprint "MountingHole:MountingHole_2mm"
 		(layer "F.Cu")
-		(at 191.07 129.39)
+		(at 199.4 106.2)
 		(descr "Mounting Hole 2mm, no annular, generated by kicad-footprint-generator mountinghole.py")
 		(tags "mountinghole")
@@
 	)
 	(via
-		(at 223.6 127.07)
+		(at 223.67 124.2)
 		(size 0.6)
 		(drill 0.3)
@@
 	)
 	(via
-		(at 221.6 125.07)
+		(at 221.67 126.2)
 		(size 0.6)
 		(drill 0.3)
@@
 	)
 	(via
-		(at 220.6 124.07)
+		(at 220.67 127.2)
 		(size 0.6)
 		(drill 0.3)
@@
 	)
 	(via
-		(at 222.6 126.07)
+		(at 222.67 125.2)
 		(size 0.6)
 		(drill 0.3)

Commit message: Add files via upload
Parts:
- SW1, SW10, SW2, SW3, SW4, SW5, SW6, SW7, SW8, SW9: footprint Button_Switch_THT:SW_PUSH_6mm -> Button_Switch_THT:SW_TH_Tactile_Omron_B3F-107x
- SW11, SW12, SW13: footprint Button_Switch_THT:SW_Tactile_SKHH_Angled -> Button_Switch_THT:SW_SPST_Omron_B3F-315x_Angled
- moved R10 4.62 mm to (216.4, 104.2)
- moved D5 3.24 mm to (95.1, 110.4)
- moved C6 2.86 mm to (191.4, 124.8)
- moved D6 2.82 mm to (82.8, 123.4)
- moved D7 2.82 mm to (72.9, 107.0)
- moved C5 2.82 mm to (79.0, 117.2)
- moved D19 2.82 mm to (196.4, 125.7)
- moved D22 2.82 mm to (76.2, 113.6)
- moved D8 2.82 mm to (82.0, 102.8)
- moved SW10 2.82 mm to (86.0, 98.1)
- moved SW5 2.82 mm to (84.9, 111.3)
- moved SW6 2.82 mm to (72.9, 123.3)
- moved SW7 2.82 mm to (61.0, 111.3)
- moved SW8 2.82 mm to (73.0, 99.3)
- moved U2 2.82 mm to (209.6, 117.8)
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Routing:
- net ROW2: track 181.6 -> 203.3 mm
- net +5V: track 368.6 -> 379.6 mm
- net COL0: track 207.3 -> 216.2 mm
- net Net-(D19-DOUT): track 57.8 -> 65.0 mm
- net JOY_R_VRx: track 68.1 -> 62.4 mm
- net COL3: track 187.4 -> 192.8 mm
- net COL2: track 168.0 -> 162.8 mm
- net Net-(Q2-B): track 5.67 -> 10.5 mm
- net M_HAP_L: track 76.1 -> 80.3 mm
- net ROW1: track 247.8 -> 252.0 mm
- net JOY_L_VRx: track 117.1 -> 121.1 mm
- net JOY_L_VRy: track 98.8 -> 102.8 mm
- net +3.3V: track 282.6 -> 286.0 mm
- net JOY_SW_R-: track 5.34 -> 8.16 mm
- net Net-(D21-DOUT): track 82.3 -> 85.1 mm
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
Commit message: Add files via upload
Parts:
- removed U1, U2: COM-09032, Joy:JOYSTICK
- added SW16: RKJXV1224005, lcsc:SW-TH_RKJXV1224005, F.Cu at (75.5, 81.0)
- added SW17: RKJXV1224005, lcsc:SW-TH_RKJXV1224005, F.Cu at (210.5, 117.0)
- SW1, SW10, SW2, SW3, SW4, SW5, SW6, SW7, SW8, SW9: value SW_Push -> B3F-1070; footprint Button_Switch_THT:SW_TH_Tactile_Omron_B3F-107x -> lcsc:SW-TH_4P-L6.2-W6.2-P4.50-LS6.5
- SW11, SW12, SW13: value SW_Push -> B3F-3152; footprint Button_Switch_THT:SW_SPST_Omron_B3F-315x_Angled -> lcsc:KEY-TH_4P-L7.3-W10.2-P4.50-LS7.0
- moved R10 5.08 mm to (218.0, 109.0)
- moved SW10 3.95 mm to (89.3, 100.3)
- moved SW3 3.95 mm to (197.6, 84.0)
- moved SW4 3.95 mm to (209.6, 72.0)
- moved SW5 3.95 mm to (88.2, 113.6)
- moved SW6 3.95 mm to (76.2, 125.6)
- moved SW7 3.95 mm to (64.2, 113.6)
- moved SW8 3.95 mm to (76.2, 101.6)
- moved SW1 3.95 mm to (221.6, 84.0)
- moved SW2 3.95 mm to (209.6, 96.0)
- moved SW9 3.95 mm to (197.6, 97.5)
- moved D14 3.53 mm to (220.0, 110.0)
- moved D16 2.97 mm to (63.5, 85.5), turned to 0 degrees
- moved SW12 2.35 mm to (66.3, 67.2), turned to 180 degrees
- moved SW13 2.35 mm to (114.9, 67.3), turned to 180 degrees
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Connections:
- D6 pad 2: Net-(D6-A) -> unconnected-(D6-A-Pad2)
- SW1 pad 2: COL1 -> Net-(D1-A)
- SW10 pad 2: COL3 -> Net-(D10-A)
- SW11 pad 2: COL0 -> Net-(D11-A)
- SW12 pad 2: COL3 -> Net-(D12-A)
- SW13 pad 2: COL3 -> Net-(D13-A)
- SW14 pad S1: COL0 -> EC11+
- SW2 pad 2: COL1 -> Net-(D2-A)
- SW3 pad 2: COL1 -> Net-(D3-A)
- SW4 pad 2: COL1 -> Net-(D4-A)
- SW5 pad 2: COL2 -> Net-(D5-A)
- SW6 pad 1: Net-(D6-A) -> unconnected-(SW6-Pad1)
- SW6 pad 2: COL2 -> unconnected-(SW6-Pad2)
- SW7 pad 2: COL2 -> Net-(D7-A)
- SW8 pad 2: COL2 -> Net-(D8-A)
- SW9 pad 2: COL0 -> Net-(D9-A)
Routing:
- net ROW1: track 252.0 -> 216.7 mm, vias 4 -> 6
- net +3.3V: track 286.0 -> 303.3 mm, vias 6 -> 5
- net JOY_L_VRx: track 121.1 -> 111.1 mm
- net Net-(D6-A): track 8.82 -> 0.00 mm
- net (no net): track 0.00 -> 8.82 mm
- net JOY_SW_L-: track 2.63 -> 10.1 mm
- net COL3: track 192.8 -> 186.1 mm, vias 1 -> 3
- net ROW2: track 203.3 -> 196.6 mm
- net Net-(D19-DOUT): track 65.0 -> 69.3 mm
- net Net-(Q2-B): track 10.5 -> 14.2 mm
- net M_HAP_R: track 94.8 -> 98.4 mm
- net JOY_L_VRy: track 102.8 -> 106.2 mm
- net JOY_SW_R-: track 8.16 -> 10.7 mm
- net M_HAP_L: track 80.3 -> 82.8 mm
- net COL2: track 162.8 -> 160.6 mm
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
Commit message: Add files via upload
Parts:
- SW14: value RotaryEncoder_Switch_MP -> EC11E09244BS; footprint Rotary_Encoder:RotaryEncoder_Alps_EC11E-Switch_Vertical_H20mm -> lcsc:SW-TH_EC11XXXXXXXX
- moved SW14 7.66 mm to (196.0, 71.2), turned to 90 degrees
- moved G*** 2.72 mm to (210.0, 117.4)
- moved D12 2.63 mm to (64.2, 72.3)
- moved SW11 0.92 mm to (220.2, 67.6)
- moved SW12 0.83 mm to (65.5, 67.5)
- moved G*** 0.64 mm to (76.2, 80.2)
- moved D11 0.55 mm to (213.8, 67.2)
Connections:
- D6 pad 2: unconnected-(D6-A-Pad2) -> Net-(D6-A)
- SW10 pad 3: JOY_SW_L+ -> COL3
- SW10 pad 4: JOY_SW_L+ -> COL3
- SW11 pad 2: Net-(D11-A) -> COL0
- SW11 pad 3: COL0 -> Net-(D11-A)
- SW11 pad 4: EC11+ -> COL0
- SW12 pad 2: Net-(D12-A) -> COL3
- SW12 pad 3: JOY_SW_L+ -> Net-(D12-A)
- SW12 pad 4: JOY_SW_L+ -> COL3
- SW13 pad 2: Net-(D13-A) -> COL3
- SW13 pad 3: COL3 -> Net-(D13-A)
- SW13 pad 4: JOY_SW_L+ -> COL3
- SW16 pad a: JOY_SW_L+ -> COL3
- SW16 pad c: JOY_SW_L+ -> COL3
- SW17 pad a: EC11+ -> COL0
- SW17 pad c: EC11+ -> COL0
- SW6 pad 1: unconnected-(SW6-Pad1) -> Net-(D6-A)
- SW6 pad 2: unconnected-(SW6-Pad2) -> Net-(D6-A)
- SW6 pad 3: unconnected-(SW6-Pad3) -> COL2
- SW6 pad 4: unconnected-(SW6-Pad4) -> COL2
- SW9 pad 3: EC11+ -> COL0
- SW9 pad 4: EC11+ -> COL0
Routing:
- net COL3: track 186.1 -> 199.1 mm
- net ROW0: track 208.0 -> 196.9 mm
- net Net-(D6-A): track 0.00 -> 8.82 mm
- net (no net): track 8.82 -> 0.00 mm
- net Net-(D12-A): track 2.94 -> 10.0 mm
- net Net-(D11-A): track 2.73 -> 9.46 mm
- net Net-(D13-A): track 5.13 -> 11.1 mm
- net ROW3: track 210.5 -> 208.4 mm
- net Net-(D20-DOUT): track 159.7 -> 158.0 mm
- net COL0: track 216.4 -> 217.4 mm
- net GND: vias 1530 -> 1766
Other:
- board text added: "Joy Controller V2.14 @Merlin2LmmL"
- board text removed: "Joy Controller V2 @Merlin2LmmL"
- board text removed: "PS5 Joystick"
