File: PCB/Joy Controller V2.kicad_sch (KiCad schematic)
At the start: 73 parts, among them J1 USB_C_Receptacle_USB2.0_16P, J2 Conn_02x16_Odd_Even, Q1 NPN, Q2 NPN, SW1 SW_Push, SW10 SW_Push, SW11 SW_Push, SW12 SW_Push, SW13 SW_Push, SW14 RotaryEncoder_Switch_MP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

Commit message: Add files via upload
Parts:
- SW1, SW10, SW2, SW3, SW4, SW5, SW6, SW7, SW8, SW9: footprint Button_Switch_THT:SW_PUSH_6mm -> Button_Switch_THT:SW_TH_Tactile_Omron_B3F-107x
- SW11, SW12, SW13: footprint Button_Switch_THT:SW_Tactile_SKHH_Angled -> Button_Switch_THT:SW_SPST_Omron_B3F-315x_Angled
Connections:
- no-connect marks 6 -> 7
Changed lines of the file:
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@@
 	)
 	(no_connect
+		(at 38.1 20.32)
+	)
+	(no_connect
 		(at 120.65 57.15)
 	)
@@
 			)
 		)
-		(property "Footprint" "Button_Switch_THT:SW_PUSH_6mm"
+		(property "Footprint" "Button_Switch_THT:SW_TH_Tactile_Omron_B3F-107x"
 			(at 266.7 133.35 0)
 			(effects
@@
 			)
 		)
-		(property "Footprint" "Button_Switch_THT:SW_Tactile_SKHH_Angled"
+		(property "Footprint" "Button_Switch_THT:SW_SPST_Omron_B3F-315x_Angled"
 			(at 266.7 102.87 0)
 			(effects
@@
 			)
 		)
-		(property "Footprint" "Button_Switch_THT:SW_Tactile_SKHH_Angled"
+		(property "Footprint" "Button_Switch_THT:SW_SPST_Omron_B3F-315x_Angled"
 			(at 185.42 102.87 0)
 			(effects
@@
 			)
 		)
-		(property "Footprint" "Button_Switch_THT:SW_PUSH_6mm"
+		(property "Footprint" "Button_Switch_THT:SW_TH_Tactile_Omron_B3F-107x"
 			(at 237.49 148.59 0)
 			(effects
@@
 			)
 		)
-		(property "Footprint" "Button_Switch_THT:SW_PUSH_6mm"
+		(property "Footprint" "Button_Switch_THT:SW_TH_Tactile_Omron_B3F-107x"
 			(at 210.82 133.35 0)
 			(effects
@@
 			)
 		)
-		(property "Footprint" "Button_Switch_THT:SW_PUSH_6mm"
+		(property "Footprint" "Button_Switch_THT:SW_TH_Tactile_Omron_B3F-107x"
 			(at 237.49 102.87 0)
 			(effects
@@
 			)
 		)
-		(property "Footprint" "Button_Switch_THT:SW_PUSH_6mm"
+		(property "Footprint" "Button_Switch_THT:SW_TH_Tactile_Omron_B3F-107x"
 			(at 210.82 118.11 0)
 			(effects
@@
 			)
 		)
-		(property "Footprint" "Button_Switch_THT:SW_PUSH_6mm"
+		(property "Footprint" "Button_Switch_THT:SW_TH_Tactile_Omron_B3F-107x"
 			(at 210.82 148.59 0)
 			(effects
@@
 			)
 		)
-		(property "Footprint" "Button_Switch_THT:SW_Tactile_SKHH_Angled"
+		(property "Footprint" "Button_Switch_THT:SW_SPST_Omron_B3F-315x_Angled"
 			(at 185.42 148.59 0)
 			(effects
@@
 			)
 		)
-		(property "Footprint" "Button_Switch_THT:SW_PUSH_6mm"
+		(property "Footprint" "Button_Switch_THT:SW_TH_Tactile_Omron_B3F-107x"
 			(at 237.49 133.35 0)
 			(effects
@@
 			)
 		)
-		(property "Footprint" "Button_Switch_THT:SW_PUSH_6mm"
+		(property "Footprint" "Button_Switch_THT:SW_TH_Tactile_Omron_B3F-107x"
 			(at 185.42 118.11 0)
 			(effects
@@
 			)
 		)
-		(property "Footprint" "Button_Switch_THT:SW_PUSH_6mm"
+		(property "Footprint" "Button_Switch_THT:SW_TH_Tactile_Omron_B3F-107x"
 			(at 237.49 118.11 0)
 			(effects
@@
 			)
 		)
-		(property "Footprint" "Button_Switch_THT:SW_PUSH_6mm"
+		(property "Footprint" "Button_Switch_THT:SW_TH_Tactile_Omron_B3F-107x"
 			(at 210.82 102.87 0)
 			(effects

Commit message: Add files via upload
Parts:
- removed SW1, SW10, SW2, SW3, SW4, SW5, SW6, SW7, SW8, SW9: SW_Push, Button_Switch_THT:SW_TH_Tactile_Omron_B3F-107x, symbol Switch:SW_Push
- removed SW11, SW12, SW13: SW_Push, Button_Switch_THT:SW_SPST_Omron_B3F-315x_Angled, symbol Switch:SW_Push
- removed U1, U2: COM-09032, Joy:JOYSTICK, symbol COM-09032:COM-09032
- added SW1, SW10, SW2, SW3, SW4, SW5, SW6, SW7, SW8, SW9: B3F-1070, lcsc:SW-TH_4P-L6.2-W6.2-P4.50-LS6.5, symbol lcsc:B3F-1070
- added SW11, SW12, SW13: B3F-3152, lcsc:KEY-TH_4P-L7.3-W10.2-P4.50-LS7.0, symbol lcsc:B3F-3152
- added SW16, SW17: RKJXV1224005, lcsc:SW-TH_RKJXV1224005, symbol lcsc:RKJXV1224005
Connections:
- net +3.3V: now also SW16.1 (B), SW16.6 (B), SW17.1 (B), SW17.6 (B)
- net COL0: now also SW11.2, SW11.4, SW17.a, SW17.c, SW9.2, SW9.3
- net COL1: now also SW1.2, SW1.3, SW2.2, SW2.3, SW3.2, SW3.3, SW4.2, SW4.3
- net COL2: now also SW5.2, SW5.3, SW7.2, SW7.3, SW8.2, SW8.3
- net COL3: now also SW13.2
- net GND: now also SW16.10 (GND), SW16.3 (A), SW16.4 (A), SW16.7 (GND), SW16.8 (GND), SW16.9 (GND), SW17.10 (GND), SW17.3 (A), SW17.4 (A), SW17.7 (GND), SW17.8 (GND), SW17.9 (GND)
- net JOY_L_VRx: now also SW16.5 (DTA)
- net JOY_L_VRy: now also SW16.2 (DTA)
- net JOY_R_VRx: now also SW17.5 (DTA)
- net JOY_R_VRy: now also SW17.2 (DTA)
- net JOY_SW_L-: now also SW16.b, SW16.d
- net JOY_SW_R-: now also SW17.b, SW17.d
- net ROW0: no longer D11.1 (K)
- net at D9.2 (A): now also SW9.1, SW9.4
- net at D11.2 (A): now also SW11.1, SW11.3
- net at D13.2 (A): now also SW13.3
- net at D4.2 (A): now also SW4.1, SW4.4
- net at D7.2 (A): now also SW7.1, SW7.4
- net at D1.2 (A): now also SW1.1, SW1.4
- net at D3.2 (A): now also SW3.1, SW3.4
- net at D6.2 (A): now also SW6.1, SW6.4
- net at D8.2 (A): now also SW8.1, SW8.4
- net at D2.2 (A): now also SW2.1, SW2.4
- net at D12.2 (A): now also SW12.1, SW12.3
- net at D10.2 (A): now also SW10.1, SW10.4
- net at D5.2 (A): now also SW5.1, SW5.4
- new net: SW6.2, SW6.3
- new net JOY_SW_L+: SW10.2, SW10.3, SW12.2, SW12.4, SW13.4, SW16.a, SW16.c
Other:
- note added: "MENU"
- note removed: "Menu"
- note removed: "SHOULDER LEFT"
- note removed: "SW"
- note removed: "VRx"
- note removed: "VRy"
- moved on the sheet: C5, C6, C7, C8, D12, D13, D19, D20, D21, D22, H1, H2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

Commit message: Add files via upload
Parts:
- removed SW14: RotaryEncoder_Switch_MP, Rotary_Encoder:RotaryEncoder_Alps_EC11E-Switch_Vertical_H20mm, symbol Device:RotaryEncoder_Switch_MP
- added SW14: EC11E09244BS, lcsc:SW-TH_EC11XXXXXXXX, symbol lcsc:EC11E09244BS
Connections:
- net COL0: now also SW9.4, SW14.E; no longer SW9.2
- net COL1: now also SW1.4, SW2.4, SW3.4, SW4.4; no longer SW1.2, SW2.2, SW3.2, SW4.2
- net COL2: now also SW5.4, SW6.3, SW6.4, SW7.4, SW8.4; no longer SW5.2, SW7.2, SW8.2
- net COL3: now also SW10.3, SW10.4, SW12.2, SW12.4, SW13.4, SW16.a, SW16.c
- net EC11-: now also SW14.D
- net GND: now also SW14.6, SW14.7, SW14.C
- net ROT_ENC_A: now also SW14.A
- net ROT_ENC_B: now also SW14.B
- net ROW0: now also D11.1 (K)
- net at D10.2 (A), SW10.1: now also SW10.2; no longer SW10.4
- net at D4.2 (A), SW4.1: now also SW4.2; no longer SW4.4
- net at D3.2 (A), SW3.1: now also SW3.2; no longer SW3.4
- net at D6.2 (A), SW6.1: now also SW6.2; no longer SW6.4
- net at D7.2 (A), SW7.1: now also SW7.2; no longer SW7.4
- net at D8.2 (A), SW8.1: now also SW8.2; no longer SW8.4
- net at D9.2 (A), SW9.1: now also SW9.2; no longer SW9.4
- net at D2.2 (A), SW2.1: now also SW2.2; no longer SW2.4
- net at D1.2 (A), SW1.1: now also SW1.2; no longer SW1.4
- net at D13.2 (A), SW13.3: now also SW13.1
- net at D5.2 (A), SW5.1: now also SW5.2; no longer SW5.4
- removed net JOY_SW_L+: SW10.2, SW10.3, SW12.2, SW12.4, SW13.4, SW16.a, SW16.c
